File: circuit/NovaBox_8635.kicad_pcb (KiCad board)
At the start: 2 copper layers, 82 x 30 mm, 87 parts, among them P1 MH, P2 MH, P3 MH, P4 MH, P5 USB, Q1 MMBT3904, Q2 IRLML6344, Q3 IRLML6401, Q4 MMBT3904, Q5 MMBT3904, SW1 PIO18, SW2 PIO21, SW3 PIO8, SW4 PIO0, SW5 PIO1, SW6 ON/OFF, U1 MCP6004, U2 CSR8635_MODULE, U3 CSR_DebugSmall, U4 PAM8304, U5 PAM8304, U6 LT1308

Commit message: sent PCB to manufacture
Parts:
- moved G*** 0.40 mm to (68.2, 73.5), turned to 270 degrees
Connections:
- net Net-(BT1-Pad2) renamed /-BATT
Routing:
- added copper zone on B.Cu, net +BATT
- added copper zone on B.Cu, net /-BATT
Other:
- board text added: "2018.aug.20"
- board text removed: "2018.aug.19"
