File: circuit/WhiteBoy.kicad_pcb (KiCad board)
At the start: 2 copper layers, 100 x 100 mm, 109 parts, among them J1 HOLE, J2 HOLE, J3 HOLE, J4 HOLE, J5 USB_B, Q1 IRF530NPbF, Q2 BC547, Q3 BC557, SW1 POS, SW2 NEG, SW3 vol+, SW4 vol-, SW5 next, SW6 prev, SW7 pause, SW8 refresh, SW9 channel, T1 PB0, T4 PC1, T5 PC3, T6 PD6, T7 PD7, U1 74AC164, U10 74AC164, U11 CSR_CFG, U12 TPA3136D2, U13 CSR8645_MODULE, U2 DS18B20, U3 MAX6457, U4 INA219_SOIC, U5 AVR-ISP6, U6 ATMEGA88PA-16AU, U7 74AC164, U8 DBG, U9 LM2576T-ADJ, Y1 16MHz

Commit message: almost done
Parts:
- added R27: 90K9, NovaBox:R_10MM, F.Cu at (67.3, 65.4)
- L1: footprint NovaBox:COIL_D9_P2.54 -> NovaBox:COIL_LHL10TB681K
- S1: value BATT_SEL -> Val
- moved C19 10.0 mm to (53.3, 114.9), turned to 90 degrees
- moved C13 10.0 mm to (53.3, 131.4), turned to 90 degrees
- moved R6 8.35 mm to (67.3, 70.5), turned to 0 degrees
- moved R11 4.62 mm to (67.3, 62.9)
- moved L2 4.62 mm to (63.5, 130.8)
- moved L3 4.62 mm to (63.5, 115.6)
- moved R10 4.62 mm to (67.3, 60.3)
- moved R4 2.29 mm to (67.3, 67.9), turned to 180 degrees
- moved L1 0.90 mm to (79.4, 92.7)
- moved S1 0.90 mm to (53.3, 64.1)
- moved C17 0.68 mm to (72.4, 127.4)
- moved BT1 0.64 mm to (69.8, 54.4)
- moved C18 0.64 mm to (72.4, 119.4)
Connections:
- S1 pad 1: Net-(R10-Pad1) -> /MAX_VDIV
- S1 pad 2: /MAX_VDIV -> Net-(R10-Pad1)
Routing:
- net /SW_GATE: track 29.0 -> 15.9 mm
- net Net-(R27-Pad1): track 0.00 -> 8.15 mm
- net +BATT: track 55.4 -> 62.5 mm
- net Net-(C19-Pad1): track 16.0 -> 11.3 mm
- net Net-(C13-Pad2): track 16.0 -> 11.4 mm
- net /OUTR: track 19.6 -> 15.6 mm
- net /OUTL: track 19.2 -> 15.5 mm
- net -BATT: track 43.9 -> 47.1 mm
- net /MAX_VDIV: track 29.5 -> 32.3 mm
- net Net-(R10-Pad1): track 9.31 -> 8.15 mm
- net Net-(D1-Pad1): track 14.8 -> 15.7 mm
- net Net-(C17-Pad2): track 12.5 -> 11.7 mm
- net Net-(C18-Pad2): track 11.0 -> 11.7 mm
Other:
- board text added: "White"
- board text added: "left"
- board text added: "right"
- board text removed: "white"

Commit message: PCB sent to production
Parts:
- added G***: , NovaBox:OSHW_18mm, B.Cu at (85.1, 58.8)
- moved L2 0.63 mm to (63.5, 131.4)
- moved L3 0.63 mm to (63.5, 114.9)
Routing:
- net Net-(C18-Pad2): track 11.7 -> 10.4 mm
- net Net-(C17-Pad2): track 11.7 -> 10.6 mm
- net /PREV: track 36.2 -> 37.0 mm
- net /OUTR: track 15.6 -> 16.3 mm
Other:
- board text added: "by Ferenc Szili https://github.com/nodep/NovaBox/ 2019.feb.04"
- board text removed: "https://github.com/nodep/NovaBox/ 2019.feb.10"
