File: circuit/WhiteBoy.kicad_pcb (KiCad board)
At the start: 2 copper layers, 100 x 100 mm, 111 parts, among them J1 HOLE, J2 HOLE, J3 HOLE, J4 HOLE, J5 USB_B, Q1 IRF530NPbF, Q2 BC547, Q3 BC557, SW1 POS, SW2 NEG, SW3 vol+, SW4 vol-, SW5 next, SW6 prev, SW7 pause, SW8 refresh, SW9 channel, T1 PB0, T4 PC1, T5 PC3, T6 PD6, T7 PD7, U1 74AC164, U10 74AC164, U11 CSR_CFG, U12 TPA3136D2, U13 CSR8645_MODULE, U2 DS18B20, U3 MAX6457, U4 INA219_SOIC, U5 AVR-ISP6, U6 ATMEGA88PA-16AU, U7 74AC164, U8 DBG, U9 LM2576T-ADJ, Y1 16MHz

Commit message: calced resistor values for battery protection on WhiteBoy
Parts:
- R10: value 115K -> 226K
- R11: value 90K9 -> 162K
- R27: value 90K9 -> 187K
- R6: value 750K -> 1M69
- S1: value Val -> BATT_SEL
Changed lines of the file:
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@@
       (effects (font (size 0.75 0.75) (thickness 0.15)))
     )
-    (fp_text value Val (at 0 -1.27) (layer F.Fab) hide
+    (fp_text value BATT_SEL (at 0 -1.27) (layer F.Fab) hide
       (effects (font (size 0.127 0.127) (thickness 0.001)))
     )
@@
       (effects (font (size 0.75 0.75) (thickness 0.15)))
     )
-    (fp_text value 90K9 (at -2.286 0) (layer F.Fab) hide
+    (fp_text value 162K (at -2.286 0) (layer F.Fab) hide
       (effects (font (size 0.127 0.127) (thickness 0.001)))
     )
@@
       (effects (font (size 0.75 0.75) (thickness 0.15)))
     )
-    (fp_text value 750K (at -2.286 0) (layer F.Fab) hide
+    (fp_text value 1M69 (at -2.286 0) (layer F.Fab) hide
       (effects (font (size 0.127 0.127) (thickness 0.001)))
     )
@@
       (effects (font (size 0.75 0.75) (thickness 0.15)))
     )
-    (fp_text value 115K (at -2.286 0) (layer F.Fab) hide
+    (fp_text value 226K (at -2.286 0) (layer F.Fab) hide
       (effects (font (size 0.127 0.127) (thickness 0.001)))
     )
@@
       (effects (font (size 0.75 0.75) (thickness 0.15)))
     )
-    (fp_text value 90K9 (at -2.286 0) (layer F.Fab) hide
+    (fp_text value 187K (at -2.286 0) (layer F.Fab) hide
       (effects (font (size 0.127 0.127) (thickness 0.001)))
     )

Commit message: SwampThing routed!
Parts:
- D2: value LED_RCBG -> LED_RABG; footprint NovaBox:LED_RCBG -> NovaBox:LED_D5.0mm_RGB
Connections:
- R14 pad 2: Net-(D2-PadGA) -> Net-(D2-Pad4)
- R15 pad 2: Net-(D2-PadBA) -> Net-(D2-Pad3)
- R17 pad 2: Net-(D2-PadRA) -> Net-(D2-Pad1)
Routing:
- net Net-(D2-PadGA): track 5.61 -> 0.00 mm
- net Net-(D2-Pad4): track 0.00 -> 5.61 mm
- net Net-(D2-PadRA): track 5.08 -> 0.00 mm
- net Net-(D2-PadBA): track 5.08 -> 0.00 mm
- net Net-(D2-Pad3): track 0.00 -> 5.08 mm
- net Net-(D2-Pad1): track 0.00 -> 5.08 mm
